File: motor_controller.kicad_sch (KiCad schematic)
At the start: 4 parts

Commit message: MCU migration completed
Other:
- title: (none) -> RBC by UGS
Changed lines of the file:
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@@
 (kicad_sch (version 20230121) (generator eeschema)
   (paper "A4")
+  (title_block
+    (title "RBC by UGS")
+    (date "2023-09-04")
+    (rev "2.0")
+  )
   (junction (at 152.4 111.76) (diameter 0) (color 0 0 0 0)
   )
