File: rbc_circuits.kicad_pcb (KiCad board)
At the start: 4 copper layers, 120 x 140 mm, 82 parts, among them IC1 BTN70301EPAXUMA1, IC2 BTN70301EPAXUMA1, IC3 BTN70301EPAXUMA1, IC4 BTN70301EPAXUMA1, IC5 BTN70301EPAXUMA1, IC6 BTN70301EPAXUMA1, IC7 BTN70301EPAXUMA1, IC8 BTN70301EPAXUMA1, J1 Conn_01x02_Pin, J2 Conn_01x02_Pin, J3 Conn_01x02_Pin, J4 Conn_01x06_Pin, J5 Conn_01x06_Pin, J6 Conn_01x02_Pin, J7 Conn_01x06_Pin, J8 Conn_01x06_Pin, J9 Conn_01x02_Pin, U1 TPS54202DDC

Commit message: PCB initial commit
Parts:
- removed A1: A000067, A000067:ARDUINO_A000067
- removed REF** (x4): MountingHole_4.3mm_M4, MountingHole:MountingHole_4.3mm_M4
- added C15: 10nF, Capacitor_SMD:C_0805_2012Metric, F.Cu at (5.36, 56.0)
- added C16: 10nF, Capacitor_SMD:C_0805_2012Metric, F.Cu at (5.36, 59.0)
- added C17: 100uF, SamacSys_Parts:16SVF180M, F.Cu at (31.2, 56.2)
- added C18: 100uF, SamacSys_Parts:16SVF180M, F.Cu at (40.9, 56.2)
- added C19: 100nF, Capacitor_SMD:C_0402_1005Metric, F.Cu at (179.7, 122.3)
- added C20: 100nF, Capacitor_SMD:C_0402_1005Metric, F.Cu at (179.7, 124.3)
- added C21: 100nF, Capacitor_SMD:C_0402_1005Metric, F.Cu at (179.7, 126.3)
- added C22: 100nF, Capacitor_SMD:C_0402_1005Metric, F.Cu at (179.7, 128.2)
- added C23: 100nF, Capacitor_SMD:C_0402_1005Metric, F.Cu at (203.2, 161.5)
- added C24: 150uF, SamacSys_Parts:EEHZT1E331UP, F.Cu at (53.2, 97.0)
- added C25: 100nF, Capacitor_SMD:C_0402_1005Metric, F.Cu at (65.9, 105.2)
- added C26: 10nF, Capacitor_SMD:C_0805_2012Metric, F.Cu at (62.3, 103.7)
- added C27: 100uF, SamacSys_Parts:16SVF180M, F.Cu at (62.7, 72.4)
- added C28: 220nF, Capacitor_SMD:C_0805_2012Metric, F.Cu at (11.7, 90.8)
- added C29: 220nF, Capacitor_SMD:C_0805_2012Metric, F.Cu at (11.7, 93.8)
- added C30: 100nF, Capacitor_SMD:C_0402_1005Metric, F.Cu at (10.9, 99.3)
- added C31: 100nF, Capacitor_SMD:C_0402_1005Metric, F.Cu at (10.9, 101.3)
- added C32: 220nF, Capacitor_SMD:C_0805_2012Metric, F.Cu at (11.7, 96.8)
- added C33: 100nF, Capacitor_SMD:C_0402_1005Metric, F.Cu at (10.9, 103.3)
- added D1: 450mV 3A, Diode_SMD:D_SMA, F.Cu at (39.2, 18.3)
- added D10: Red, Diode_SMD:D_0805_2012Metric, F.Cu at (40.5, 101.6)
- added D2: 450mV 3A, Diode_SMD:D_SMA, F.Cu at (39.2, 22.9)
- added D3: 450mV 3A, Diode_SMD:D_SMA, F.Cu at (39.2, 27.4)
- added D4: LED, Diode_SMD:D_0805_2012Metric, F.Cu at (193.6, 130.7)
- added D5: 450mV 3A, Diode_SMD:D_SMA, F.Cu at (71.6, 75.6)
- added D6: Green, Diode_SMD:D_0805_2012Metric, F.Cu at (40.5, 89.4)
- added D7: Green, Diode_SMD:D_0805_2012Metric, F.Cu at (40.5, 92.5)
- added D8: Green, Diode_SMD:D_0805_2012Metric, F.Cu at (40.5, 95.5)
- added D9: Green, Diode_SMD:D_0805_2012Metric, F.Cu at (40.5, 98.6)
- added IC10: BTN70301EPAXUMA1, rbc Custom Library:Infineon_PG-TSDSO-14-22_custom, F.Cu at (-9.50, 95.3)
- added IC11: BTN70301EPAXUMA1, rbc Custom Library:Infineon_PG-TSDSO-14-22_custom, F.Cu at (-9.50, 101.7)
- added IC9: BTN70301EPAXUMA1, rbc Custom Library:Infineon_PG-TSDSO-14-22_custom, F.Cu at (-9.50, 88.8)
- added J10: Conn_01x06_Pin, Connector_Molex:Molex_Micro-Fit_3.0_43045-0612_2x03_P3.00mm_Vertical, F.Cu at (-0.87, 80.6)
- added J11: Conn_01x06_Pin, Connector_Molex:Molex_Micro-Fit_3.0_43045-0612_2x03_P3.00mm_Vertical, F.Cu at (-0.87, 91.4)
- added JP3: ON, Jumper:SolderJumper-2_P1.3mm_Open_RoundedPad1.0x1.5mm, F.Cu at (69.7, 71.6)
- added L2: 22uH, SamacSys_Parts:INDPM110100X400N, F.Cu at (-6.76, 22.0)
- added L3: 22uH, SamacSys_Parts:INDPM110100X400N, F.Cu at (-6.76, 33.8)
- added L4: 22uH, SamacSys_Parts:INDPM110100X400N, F.Cu at (-6.76, 45.7)
- added L5: 10uH, Inductor_SMD:L_0805_2012Metric, F.Cu at (194.3, 125.7)
- added L6: 22uH, SamacSys_Parts:INDPM110100X400N, F.Cu at (52.6, 85.4)
- added R43: 4k7, Resistor_SMD:R_1206_3216Metric, F.Cu at (23.5, 77.8)
- added R44: 4k7, Resistor_SMD:R_1206_3216Metric, F.Cu at (23.5, 81.1)
- added R45: 4k7, Resistor_SMD:R_1206_3216Metric, F.Cu at (23.5, 84.4)
- added R46: 1k2, Resistor_SMD:R_1206_3216Metric, F.Cu at (23.5, 87.7)
- added R47: 4k7, Resistor_SMD:R_1206_3216Metric, F.Cu at (29.1, 67.9)
- added R48: 4k7, Resistor_SMD:R_1206_3216Metric, F.Cu at (29.1, 71.2)
- added R49: 4k7, Resistor_SMD:R_1206_3216Metric, F.Cu at (29.1, 74.5)
- added R50: 4k7, Resistor_SMD:R_1206_3216Metric, F.Cu at (29.1, 77.8)
- added R51: 4k7, Resistor_SMD:R_1206_3216Metric, F.Cu at (29.1, 81.1)
- added R52: 4k7, Resistor_SMD:R_1206_3216Metric, F.Cu at (29.1, 84.4)
- added SW1: RESET, Connector_PinHeader_2.54mm:PinHeader_1x02_P2.54mm_Vertical, F.Cu at (183.4, 123.7)
- added U2: ATmega2560-16A, Package_QFP:TQFP-100_14x14mm_P0.5mm, F.Cu at (200.0, 150.0)
- C1: value 10uF -> 1uF; footprint Capacitor_SMD:C_1206_3216Metric_Pad1.33x1.80mm_HandSolder -> Capacitor_SMD:C_0603_1608Metric
- C10: value 100nF -> 100uF; footprint Capacitor_SMD:C_0603_1608Metric_Pad1.08x0.95mm_HandSolder -> SamacSys_Parts:16SVF180M
- C11, C12: value 220pF -> 150uF; footprint Capacitor_SMD:C_0402_1005Metric_Pad0.74x0.62mm_HandSolder -> SamacSys_Parts:EEHZT1E331UP
- C13, C14: footprint Capacitor_SMD:C_0603_1608Metric_Pad1.08x0.95mm_HandSolder -> Capacitor_SMD:C_0402_1005Metric
- C2: value 0.1uF -> 150uF; footprint Capacitor_SMD:C_0603_1608Metric_Pad1.08x0.95mm_HandSolder -> SamacSys_Parts:EEHZT1E331UP
- C3: value 0.1uF -> 4.7uF; footprint Capacitor_SMD:C_0603_1608Metric_Pad1.08x0.95mm_HandSolder -> Capacitor_SMD:C_1206_3216Metric
- C4: value 22uF -> 10nF; footprint Capacitor_SMD:C_1206_3216Metric_Pad1.33x1.80mm_HandSolder -> Capacitor_SMD:C_0402_1005Metric
- C5: value 22uF -> 100nF; footprint Capacitor_SMD:C_1206_3216Metric_Pad1.33x1.80mm_HandSolder -> Capacitor_SMD:C_0402_1005Metric
- C6: value 75pF -> 100nF; footprint Capacitor_SMD:C_0805_2012Metric_Pad1.18x1.45mm_HandSolder -> Capacitor_SMD:C_0402_1005Metric
- C7: value 220pF -> 10pF; footprint Capacitor_SMD:C_0402_1005Metric_Pad0.74x0.62mm_HandSolder -> Capacitor_SMD:C_0603_1608Metric
- C8: value 220pF -> 10nF; footprint Capacitor_SMD:C_0402_1005Metric_Pad0.74x0.62mm_HandSolder -> Capacitor_SMD:C_0805_2012Metric
- C9: value 100nF -> 22uF; footprint Capacitor_SMD:C_0603_1608Metric_Pad1.08x0.95mm_HandSolder -> Capacitor_SMD:C_1206_3216Metric
- IC1: value BTN70301EPAXUMA1 -> LT8609AEDDM#PBF; footprint rbc Custom Library:Infineon_PG-TSDSO-14-22_custom -> SamacSys_Parts:SON50P300X300X80-11N-D
- IC2, IC3, IC4, IC5: value BTN70301EPAXUMA1 -> LM2678SX-ADJ/NOPB; footprint rbc Custom Library:Infineon_PG-TSDSO-14-22_custom -> SamacSys_Parts:KTW0007B
- J2: value Conn_01x02_Pin -> Extra; footprint Connector_PinHeader_2.54mm:PinHeader_1x02_P2.54mm_Vertical -> Connector_PinHeader_2.54mm:PinHeader_2x02_P2.54mm_Vertical
- J3: value Conn_01x02_Pin -> ICSP; footprint Connector_PinHeader_2.54mm:PinHeader_1x02_P2.54mm_Vertical -> Connector_PinHeader_2.54mm:PinHeader_2x02_P2.54mm_Vertical
- J4: value Conn_01x06_Pin -> PROG; footprint Connector_Molex:Molex_Micro-Fit_3.0_43045-0612_2x03_P3.00mm_Vertical -> Connector_PinHeader_2.54mm:PinHeader_2x02_P2.54mm_Vertical
- J5: value Conn_01x06_Pin -> External Switch; footprint Connector_Molex:Molex_Micro-Fit_3.0_43045-0612_2x03_P3.00mm_Vertical -> TerminalBlock_Phoenix:TerminalBlock_Phoenix_MKDS-3-2-5.08_1x02_P5.08mm_Horizontal
- J6: value Conn_01x02_Pin -> Raspberry Pi Power/UART; footprint TerminalBlock_Phoenix:TerminalBlock_Phoenix_MKDS-3-2-5.08_1x02_P5.08mm_Horizontal -> Connector_Molex:Molex_Micro-Fit_3.0_43045-0612_2x03_P3.00mm_Vertical
- J7, J8: value Conn_01x06_Pin -> Extra 12V; footprint Connector_Molex:Molex_Micro-Fit_3.0_43045-0612_2x03_P3.00mm_Vertical -> Connector_Molex:Molex_Micro-Fit_3.0_43045-0412_2x02_P3.00mm_Vertical
- J9: value Conn_01x02_Pin -> Conn_01x06_Pin; footprint TerminalBlock_Phoenix:TerminalBlock_Phoenix_MKDS-3-2-5.08_1x02_P5.08mm_Horizontal -> Connector_Molex:Molex_Micro-Fit_3.0_43045-0612_2x03_P3.00mm_Vertical
- JP1: value SolderJumper_2_Open -> EN; footprint Jumper:SolderJumper-2_P1.3mm_Open_RoundedPad1.0x1.5mm -> Jumper:SolderJumper-3_P2.0mm_Open_TrianglePad1.0x1.5mm
- JP2: value D3087-98 -> SolderJumper_2_Open; footprint SamacSys_Parts:D308798 -> Jumper:SolderJumper-2_P1.3mm_Open_RoundedPad1.0x1.5mm
- L1: value 15uH -> 2.2uH; footprint LQH3NPH150MMEL:IND_LQH3NPH150MMEL -> SamacSys_Parts:INDC4441X200N
- R1: value 510k -> 18.2k; footprint Resistor_SMD:R_0805_2012Metric_Pad1.20x1.40mm_HandSolder -> Resistor_SMD:R_0603_1608Metric_Pad0.98x0.95mm_HandSolder
- R10, R20, R9: value 4k7 -> 8.87k; footprint Resistor_SMD:R_1206_3216Metric_Pad1.30x1.75mm_HandSolder -> Resistor_SMD:R_0603_1608Metric
- R11: value 1k2 -> 10k; footprint Resistor_SMD:R_1206_3216Metric_Pad1.30x1.75mm_HandSolder -> Resistor_SMD:R_0402_1005Metric
- R12: value 1k2 -> 1M; footprint Resistor_SMD:R_1206_3216Metric_Pad1.30x1.75mm_HandSolder -> Resistor_SMD:R_0402_1005Metric
- R13: value 4k7 -> 1k6; footprint Resistor_SMD:R_1206_3216Metric_Pad1.30x1.75mm_HandSolder -> Resistor_SMD:R_0805_2012Metric_Pad1.20x1.40mm_HandSolder
- R14: value 4k7 -> 3k3
- R15, R21, R22, R23, R24, R25: value 4k7 -> 300; footprint Resistor_SMD:R_1206_3216Metric_Pad1.30x1.75mm_HandSolder -> Resistor_SMD:R_0603_1608Metric_Pad0.98x0.95mm_HandSolder
- R16: value 4k7 -> 82k ±1%; footprint Resistor_SMD:R_1206_3216Metric_Pad1.30x1.75mm_HandSolder -> Resistor_SMD:R_0603_1608Metric_Pad0.98x0.95mm_HandSolder
- R17: value 4k7 -> 18k ±5%; footprint Resistor_SMD:R_1206_3216Metric_Pad1.30x1.75mm_HandSolder -> Resistor_SMD:R_0603_1608Metric_Pad0.98x0.95mm_HandSolder
- R18, R7, R8: value 4k7 -> 1k; footprint Resistor_SMD:R_1206_3216Metric_Pad1.30x1.75mm_HandSolder -> Resistor_SMD:R_0201_0603Metric
- R19: value 4k7 -> 10k; footprint Resistor_SMD:R_1206_3216Metric_Pad1.30x1.75mm_HandSolder -> Resistor_SMD:R_0402_1005Metric
- R2: value 49.9 -> 1k; footprint Resistor_SMD:R_0805_2012Metric_Pad1.20x1.40mm_HandSolder -> Resistor_SMD:R_0201_0603Metric
- R26, R27, R28, R30, R32, R33, R34, R35, R36, R37, R38, R39, R40, R41, R42: footprint Resistor_SMD:R_1206_3216Metric_Pad1.30x1.75mm_HandSolder -> Resistor_SMD:R_1206_3216Metric
- R29: value 1k2 -> 4k7; footprint Resistor_SMD:R_1206_3216Metric_Pad1.30x1.75mm_HandSolder -> Resistor_SMD:R_1206_3216Metric
- R3: value 100k -> 187k; footprint Resistor_SMD:R_1206_3216Metric_Pad1.30x1.75mm_HandSolder -> Resistor_SMD:R_0603_1608Metric
- R31: value 4k7 -> 1k2; footprint Resistor_SMD:R_1206_3216Metric_Pad1.30x1.75mm_HandSolder -> Resistor_SMD:R_1206_3216Metric
- R4: value 13.3k -> 8.87k; footprint Resistor_SMD:R_0805_2012Metric_Pad1.20x1.40mm_HandSolder -> Resistor_SMD:R_0603_1608Metric
- R5: value 1k6 -> 1M; footprint Resistor_SMD:R_0805_2012Metric_Pad1.20x1.40mm_HandSolder -> Resistor_SMD:R_0402_1005Metric
- R6: value 3k3 -> 100k; footprint Resistor_SMD:R_1206_3216Metric_Pad1.30x1.75mm_HandSolder -> Resistor_SMD:R_0201_0603Metric
- U1: value TPS54202DDC -> CSTCE16M0V53-R0; footprint Package_TO_SOT_SMD:SOT-23-6 -> SamacSys_Parts:CSTCE16M0V53R0
- moved J2 167.7 mm to (9.91, 53.8), turned to 0 degrees
- moved IC6 161.8 mm to (-9.50, 69.5)
- moved IC8 161.4 mm to (-9.50, 82.4)
- moved J9 160.5 mm to (-0.87, 69.8), turned to 0 degrees
- moved IC7 159.4 mm to (-9.50, 75.9)
- moved R5 158.0 mm to (-5.38, 55.1), turned to 0 degrees
- moved C14 156.2 mm to (1.70, 60.3), turned to 0 degrees
- moved J4 155.1 mm to (180.8, 151.4)
- moved R6 150.3 mm to (44.4, 18.7), turned to 0 degrees
- moved C13 149.6 mm to (1.70, 58.4), turned to 0 degrees
- moved R12 143.2 mm to (205.0, 158.1), turned to -135 degrees
- moved C1 140.5 mm to (33.1, 17.3), turned to 0 degrees
- moved C2 136.7 mm to (24.2, 21.7), turned to 0 degrees
- moved R2 133.3 mm to (44.4, 16.9), turned to 0 degrees
- moved U1 132.8 mm to (207.1, 160.2), turned to -135 degrees
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Connections:
- C1 pad 1: +BATT -> GND
- C1 pad 2: GND -> Net-(IC1-INTVCC)
- C10 pad 1: GND -> +12C
- C10 pad 2: +12V -> GND
- C11 pad 1: 4_IS -> +BATT
- C12 pad 1: 3_IS -> +BATT
- C13 pad 2: +12P -> +BATT
- C14 pad 2: +12P -> +BATT
- C3 pad 1: Net-(U1-BOOT) -> GND
- C3 pad 2: Net-(U1-SW) -> +BATT
- C4 pad 1: +5V -> GND
- C4 pad 2: GND -> Net-(IC1-TR/SS)
- C5 pad 1: +5V -> GND
- C5 pad 2: GND -> +BATT
- C6 pad 1: Net-(C6-Pad1) -> Net-(IC1-BST)
- C6 pad 2: Net-(U1-FB) -> Net-(IC1-SW)
- C7 pad 1: 1_IS -> Net-(IC1-FB)
- C7 pad 2: GND -> Net-(JP1-C)
- C8 pad 1: 2_IS -> Net-(D1-K)
- C8 pad 2: GND -> Net-(IC2-CB)
- C9 pad 1: +12V -> GND
- C9 pad 2: GND -> Net-(JP1-C)
- IC1 pad 1: unconnected-(IC1-NC_1-Pad1) -> Net-(IC1-BST)
- IC1 pad 10: 1_LOUT -> +BATT
- IC1 pad 11: unconnected-(IC1-NC_4-Pad11) -> GND
- IC1 pad 2: Net-(IC1-EN) -> Net-(IC1-SW)
- IC1 pad 3: Net-(IC1-DEN) -> Net-(IC1-INTVCC)
- IC1 pad 4: Net-(IC1-IS) -> Net-(IC1-RT)
- IC1 pad 5: unconnected-(IC1-NC_2-Pad5) -> Net-(IC1-INTVCC)
- IC1 pad 6: Net-(IC1-IN) -> Net-(IC1-FB)
- IC1 pad 7: unconnected-(IC1-NC_3-Pad7) -> Net-(IC1-TR/SS)
- IC1 pad 8: 1_LOUT -> Net-(IC1-PG)
- IC1 pad 9: 1_LOUT -> +BATT
- IC2 pad 1: unconnected-(IC2-NC_1-Pad1) -> Net-(D1-K)
- IC2 pad 2: Net-(IC2-EN) -> +BATT
- IC2 pad 3: Net-(IC2-DEN) -> Net-(IC2-CB)
- IC2 pad 4: Net-(IC2-IS) -> GND
- IC2 pad 6: Net-(IC2-IN) -> Net-(IC2-FB)
- IC2 pad 8: 2_LOUT -> unconnected-(IC2-TAB-Pad8)
- IC3 pad 1: unconnected-(IC3-NC_1-Pad1) -> Net-(D2-K)
- IC3 pad 2: Net-(IC3-EN) -> +BATT
- IC3 pad 3: Net-(IC3-DEN) -> Net-(IC3-CB)
- IC3 pad 4: Net-(IC1-IS) -> GND
- IC3 pad 6: Net-(IC3-IN) -> Net-(IC3-FB)
- IC3 pad 8: 1_ROUT -> unconnected-(IC3-TAB-Pad8)
- IC4 pad 1: unconnected-(IC4-NC_1-Pad1) -> Net-(D3-K)
- IC4 pad 2: Net-(IC4-EN) -> +BATT
- IC4 pad 3: Net-(IC4-DEN) -> Net-(IC4-CB)
- IC4 pad 4: Net-(IC2-IS) -> GND
- IC4 pad 6: Net-(IC4-IN) -> Net-(IC4-FB)
- IC4 pad 8: 2_ROUT -> unconnected-(IC4-TAB-Pad8)
- IC5 pad 1: unconnected-(IC5-NC_1-Pad1) -> Net-(D5-K)
- IC5 pad 2: Net-(IC5-EN) -> +BATT
- IC5 pad 3: Net-(IC5-DEN) -> Net-(IC5-CB)
- IC5 pad 4: Net-(IC5-IS) -> GND
- IC5 pad 6: Net-(IC5-IN) -> Net-(IC5-FB)
- IC5 pad 7: unconnected-(IC5-NC_3-Pad7) -> Net-(IC5-ON/~{OFF})
- IC5 pad 8: 4_LOUT -> unconnected-(IC5-TAB-Pad8)
- IC6 pad 10: 3_LOUT -> 1_LOUT
- IC6 pad 15: +12P -> +12V
- IC6 pad 8: 3_LOUT -> 1_LOUT
- IC6 pad 9: 3_LOUT -> 1_LOUT
- IC7 pad 10: 4_ROUT -> 2_LOUT
- IC7 pad 15: +12P -> +12C
- IC7 pad 4: Net-(IC5-IS) -> Net-(IC7-IS)
- IC7 pad 8: 4_ROUT -> 2_LOUT
- IC7 pad 9: 4_ROUT -> 2_LOUT
- IC8 pad 10: 3_ROUT -> 1_ROUT
- IC8 pad 15: +12P -> +12V
- IC8 pad 8: 3_ROUT -> 1_ROUT
- IC8 pad 9: 3_ROUT -> 1_ROUT
- J1 pad 1: Net-(J1-Pin_1) -> +BATT
- J2 pad 2: GND -> +5V
- J3 pad 1: PI_TX -> /MCU/MISO
- J3 pad 2: PI_RX -> /MCU/SCK
- J4 pad 1: 1_HALL_A -> /MCU/DTR
- J4 pad 2: +5V -> /MCU/PROG_RX
- J4 pad 3: 1_HALL_B -> /MCU/PROG_TX
- J4 pad 4: 1_LOUT -> EXTRA_A
- J5 pad 1: 2_HALL_A -> +5V
- J5 pad 2: +5V -> STOP
- J6 pad 1: +12V -> +5V
- J6 pad 2: GND -> +5V
- J7 pad 1: 4_HALL_A -> +12LF
- J7 pad 2: +5V -> +12LF
- J7 pad 3: 4_HALL_B -> GND
- J7 pad 4: 4_LOUT -> GND
- J8 pad 1: 3_HALL_A -> +12LF
- J8 pad 2: +5V -> +12LF
- J8 pad 3: 3_HALL_B -> GND
- J8 pad 4: 3_LOUT -> GND
- J9 pad 1: +12P -> 1_HALL_A
- J9 pad 2: GND -> +5V
- JP1 pad 1: Net-(JP1-A) -> +5V
- JP1 pad 2: Net-(JP1-B) -> Net-(JP1-C)
- JP2 pad 1: Net-(J1-Pin_1) -> BATT_LVL
- JP2 pad 2: +BATT -> Net-(JP2-B)
- L1 pad 1: Net-(U1-SW) -> Net-(IC1-SW)
- L1 pad 2: +5V -> Net-(JP1-C)
- R1 pad 1: +BATT -> Net-(IC1-RT)
- R1 pad 2: Net-(JP1-A) -> GND
- R10 pad 1: Net-(IC2-IS) -> +12P
- R10 pad 2: Net-(R10-Pad2) -> Net-(IC4-FB)
- R11 pad 1: GND -> +5V
- R11 pad 2: Net-(IC1-IS) -> /MCU/RESET
- R12 pad 1: GND -> Net-(U1-OUTPUT)
- R12 pad 2: Net-(IC2-IS) -> Net-(U1-INPUT)
- R13 pad 1: 1_LPWM -> Net-(U2-PJ1)
- R13 pad 2: Net-(IC1-IN) -> PI_RX
- R14 pad 1: +5V -> PI_RX
- R14 pad 2: Net-(IC1-DEN) -> GND
- R15 pad 1: +5V -> Net-(U2-PB7)
- R15 pad 2: Net-(IC1-EN) -> Net-(D4-A)
- R16 pad 1: 2_LPWM -> +BATT
- R16 pad 2: Net-(IC2-IN) -> Net-(JP2-B)
- R17 pad 1: +5V -> BATT_LVL
- R17 pad 2: Net-(IC2-DEN) -> GND
- R18 pad 1: +5V -> Net-(IC5-FB)
- R18 pad 2: Net-(IC2-EN) -> GND
- R19 pad 1: 1_RPWM -> STOP
- R19 pad 2: Net-(IC3-IN) -> GND
- R2 pad 1: +5V -> Net-(IC2-FB)
- R2 pad 2: Net-(C6-Pad1) -> GND
- R20 pad 1: Net-(IC3-DEN) -> +12LF
- R20 pad 2: +5V -> Net-(IC5-FB)
- R21 pad 1: Net-(IC3-EN) -> 5_BATT_IND
- R21 pad 2: +5V -> Net-(D6-A)
- R22 pad 1: 2_RPWM -> 4_BATT_IND
- R22 pad 2: Net-(IC4-IN) -> Net-(D7-A)
- R23 pad 1: Net-(IC4-DEN) -> 3_BATT_IND
- R23 pad 2: +5V -> Net-(D8-A)
- R24 pad 1: Net-(IC4-EN) -> 2_BATT_IND
- R24 pad 2: +5V -> Net-(D9-A)
- R25 pad 1: Net-(R25-Pad1) -> 1_BATT_IND
- R25 pad 2: 4_IS -> Net-(D10-A)
- R26 pad 2: 3_IS -> 1_IS
- R27 pad 1: Net-(IC5-IS) -> Net-(R27-Pad1)
- R27 pad 2: Net-(R25-Pad1) -> 2_IS
- R29 pad 1: GND -> Net-(IC7-IS)
- R29 pad 2: Net-(IC5-IS) -> Net-(R27-Pad1)
- R3 pad 1: Net-(C6-Pad1) -> Net-(IC1-FB)
- R3 pad 2: Net-(U1-FB) -> GND
- R31 pad 1: 4_LPWM -> GND
- R31 pad 2: Net-(IC5-IN) -> Net-(IC7-IS)
- R32 pad 1: +5V -> 1_LPWM
- R32 pad 2: Net-(IC5-DEN) -> Net-(IC6-IN)
- R33 pad 1: +5V -> M_EN_DEN
- R33 pad 2: Net-(IC5-EN) -> Net-(IC6-DEN)
- R34 pad 1: 3_LPWM -> M_EN_DEN
- R34 pad 2: Net-(IC6-IN) -> Net-(IC6-EN)
- R35 pad 1: +5V -> 2_LPWM
- R35 pad 2: Net-(IC6-DEN) -> Net-(IC7-IN)
- R36 pad 1: +5V -> M_EN_DEN
- R36 pad 2: Net-(IC6-EN) -> Net-(IC7-DEN)
- R37 pad 1: 4_RPWM -> M_EN_DEN
- R37 pad 2: Net-(IC7-IN) -> Net-(IC7-EN)
- R38 pad 1: Net-(IC7-DEN) -> 1_RPWM
- R38 pad 2: +5V -> Net-(IC8-IN)
- R39 pad 1: Net-(IC7-EN) -> Net-(IC8-DEN)
- R39 pad 2: +5V -> M_EN_DEN
- R4 pad 1: Net-(U1-FB) -> +12C
- R4 pad 2: GND -> Net-(IC2-FB)
- R40 pad 1: 3_RPWM -> Net-(IC8-EN)
- R40 pad 2: Net-(IC8-IN) -> M_EN_DEN
- R41 pad 1: Net-(IC8-DEN) -> 2_RPWM
- R41 pad 2: +5V -> Net-(IC9-IN)
- R42 pad 1: Net-(IC8-EN) -> Net-(IC9-DEN)
- R42 pad 2: +5V -> M_EN_DEN
- R5 pad 1: Net-(A1-Pad14) -> Net-(JP1-C)
- R5 pad 2: PI_RX -> Net-(IC1-FB)
- R6 pad 1: PI_RX -> Net-(JP1-C)
- R6 pad 2: GND -> Net-(IC1-PG)
- R7 pad 1: Net-(R7-Pad1) -> Net-(IC3-FB)
- R7 pad 2: 1_IS -> GND
- R8 pad 1: Net-(R10-Pad2) -> Net-(IC4-FB)
- R8 pad 2: 2_IS -> GND
- R9 pad 1: Net-(IC1-IS) -> +12V
- R9 pad 2: Net-(R7-Pad1) -> Net-(IC3-FB)
- U1 pad 1: GND -> Net-(U1-INPUT)
- U1 pad 2: Net-(U1-SW) -> GND
- U1 pad 3: +BATT -> Net-(U1-OUTPUT)
Routing:
- net 1_HALL_B: track 113.2 -> 0.00 mm, vias 2 -> 0
- net 1_HALL_A: track 108.3 -> 0.00 mm, vias 2 -> 0
- net 4_HALL_B: track 96.7 -> 0.00 mm, vias 2 -> 0
- net 2_HALL_B: track 93.5 -> 0.00 mm
- net 4_HALL_A: track 87.9 -> 0.00 mm, vias 2 -> 0
- net 2_HALL_A: track 83.4 -> 0.00 mm, vias 1 -> 0
- net 1_LPWM: track 64.0 -> 0.00 mm
- net 2_RPWM: track 62.9 -> 0.00 mm, vias 1 -> 0
- net 1_RPWM: track 62.7 -> 0.00 mm
- net 2_LPWM: track 61.7 -> 0.00 mm, vias 1 -> 0
- net 4_IS: track 59.3 -> 0.00 mm, vias 1 -> 0
- net PI_TX: track 59.2 -> 0.00 mm
- net 3_HALL_B: track 58.3 -> 0.00 mm, vias 1 -> 0
- net 3_IS: track 57.1 -> 0.00 mm, vias 3 -> 0
- net 3_RPWM: track 56.0 -> 0.00 mm, vias 1 -> 0
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- removed copper zone on B.Cu, net +12P
- removed copper zone on F.Cu, net +12P
- removed copper zone on B.Cu, net +12V
- removed copper zone on F.Cu, net +12V
- removed copper zone on F.Cu, net +5V
- removed copper zone on In2.Cu, net +5V
- removed copper zone on F.Cu, net +BATT
- removed copper zone on F.Cu, net 1_IS
- removed copper zone on F.Cu, net 1_LOUT
- removed copper zone on F.Cu, net 1_ROUT
- removed copper zone on F.Cu, net 2_IS
- removed copper zone on F.Cu, net 2_LOUT
- removed copper zone on F.Cu, net 2_ROUT
- removed copper zone on F.Cu, net 3_LOUT
- removed copper zone on F.Cu, net 3_ROUT
- removed copper zone on F.Cu, net 4_LOUT
- removed copper zone on F.Cu, net 4_ROUT
- removed copper zone on F.Cu, net GND
- removed copper zone on In1.Cu, net GND
- removed copper zone on F.Cu, net Net-(C6-Pad1)
- removed copper zone on F.Cu, net Net-(J1-Pin_1)
- removed copper zone on F.Cu, net Net-(U1-FB)
- removed copper zone on B.Cu, net Net-(U1-SW)
- removed copper zone on F.Cu, net Net-(U1-SW)
Other:
- board size 120 x 140 mm -> 200 x 200 mm
- board text removed: "MOTOR CONTROLLER PCB Rev 1.0"
- board text removed: "PROJECT RBC"
- board text removed: "© UGS 2023"

Commit message: MCU routing completed
Parts:
- removed SW1: RESET, Connector_PinHeader_2.54mm:PinHeader_1x02_P2.54mm_Vertical
- added S1: RESET, SamacSys_Parts:FSM4JSMATR, F.Cu at (210.3, 171.2)
- moved L1 273.1 mm to (202.2, 226.1), turned to 90 degrees
- moved IC1 272.7 mm to (206.8, 231.1)
- moved JP1 266.4 mm to (225.8, 218.2)
- moved C6 266.1 mm to (203.7, 229.6), turned to 180 degrees
- moved C9 258.7 mm to (187.5, 228.6)
- moved C1 254.6 mm to (203.6, 206.4)
- moved C7 254.6 mm to (203.6, 208.9)
- moved R3 254.6 mm to (203.6, 211.4)
- moved C3 251.3 mm to (184.7, 216.8)
- moved C4 251.3 mm to (197.4, 210.1)
- moved R1 251.3 mm to (191.0, 210.5)
- moved R5 251.3 mm to (190.3, 212.7)
- moved R6 250.9 mm to (206.9, 209.8)
- moved J3 48.4 mm to (180.8, 157.7), turned to 90 degrees
- moved R15 42.3 mm to (200.1, 164.8), turned to 180 degrees
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Connections:
- C22 pad 1: +5V -> Net-(U2-AVCC)
- L5 pad 2: GND -> Net-(U2-AVCC)
- U2 pad 100: +5V -> Net-(U2-AVCC)
Routing:
- net /MCU/RESET: track 3.27 -> 47.1 mm, vias 0 -> 1
- net GND: track 0.00 -> 23.9 mm, vias 0 -> 6
- net +5V: track 0.00 -> 19.4 mm
- net /MCU/SCK: track 0.00 -> 19.3 mm
- net /MCU/MOSI: track 0.00 -> 18.3 mm
- net /MCU/MISO: track 0.00 -> 18.2 mm
- net Net-(U2-AVCC): track 0.00 -> 5.74 mm
- net Net-(U2-PB7): track 0.00 -> 5.23 mm
- net Net-(D4-A): track 0.00 -> 2.07 mm
- net Net-(U1-OUTPUT): track 4.87 -> 6.88 mm
- net Net-(U1-INPUT): track 4.83 -> 6.77 mm
- added copper zone on In1.Cu, net GND

Commit message: completed 5V regulator routing
Parts:
- moved C13 191.4 mm to (186.0, 109.8)
- moved C15 191.4 mm to (189.7, 107.4)
- moved C11 189.6 mm to (204.4, 92.0)
- moved IC3 189.6 mm to (192.3, 87.6)
- moved L3 189.6 mm to (173.5, 92.8)
- moved R7 189.6 mm to (224.6, 79.4)
- moved R9 189.6 mm to (213.3, 86.3)
- moved D2 189.6 mm to (219.4, 81.8)
- moved C17 183.9 mm to (207.0, 110.2)
- moved R21 181.4 mm to (212.7, 135.7), turned to 90 degrees
- moved D6 177.4 mm to (212.7, 132.2), turned to -90 degrees
- moved R22 174.7 mm to (206.3, 135.7), turned to 90 degrees
- moved D7 170.5 mm to (206.3, 132.2), turned to -90 degrees
- moved R23 167.9 mm to (200.0, 135.7), turned to 90 degrees
- moved D8 163.7 mm to (200.0, 132.2), turned to -90 degrees
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Routing:
- net 5_BATT_IND: track 0.00 -> 12.8 mm
- net 1_BATT_IND: track 0.00 -> 12.8 mm
- net Net-(IC1-TR/SS): track 0.00 -> 7.16 mm
- net 4_BATT_IND: track 0.00 -> 6.70 mm
- net 2_BATT_IND: track 0.00 -> 6.61 mm
- net Net-(IC1-FB): track 0.00 -> 6.30 mm
- net Net-(IC1-RT): track 0.00 -> 5.15 mm, vias 0 -> 2
- net 3_BATT_IND: track 0.00 -> 4.66 mm
- net Net-(JP1-C): track 0.00 -> 4.06 mm, vias 0 -> 4
- net Net-(IC1-PG): track 0.00 -> 2.94 mm
- net Net-(D8-A): track 0.00 -> 1.71 mm
- net Net-(D7-A): track 0.00 -> 1.71 mm
- net Net-(D6-A): track 0.00 -> 1.71 mm
- net Net-(D9-A): track 0.00 -> 1.68 mm
- net Net-(D10-A): track 0.00 -> 1.66 mm
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- added copper zone on F.Cu, net +5V
- added copper zone on F.Cu, net +BATT
- added copper zone on B.Cu, net GND
- added copper zone on F.Cu, net Net-(IC1-INTVCC)
- added copper zone on F.Cu, net Net-(IC1-SW)
- added copper zone on F.Cu, net Net-(JP1-C)
- added copper zone on In2.Cu, net Net-(JP1-C)

Commit message: completed 12 V regulators routing
Parts:
- C11, C12, C2, C24: value 150uF -> 270uF; footprint SamacSys_Parts:EEHZT1E331UP -> SamacSys_Parts:EEHZS1H221P
- IC2, IC3, IC4, IC5: footprint SamacSys_Parts:KTW0007B -> rbc Custom Library:KTW0007B_custom
- moved L4 294.3 mm to (262.2, 165.1), turned to 180 degrees
- moved IC4 288.6 mm to (278.1, 152.5), turned to -90 degrees
- moved C16 281.8 mm to (269.1, 158.2)
- moved L2 278.2 mm to (254.3, 118.0), turned to 180 degrees
- moved R10 276.2 mm to (275.1, 163.0), turned to 90 degrees
- moved IC2 272.9 mm to (270.3, 105.5), turned to -90 degrees
- moved D3 269.3 mm to (271.3, 164.1), turned to 90 degrees
- moved C14 267.7 mm to (253.1, 152.4), turned to -90 degrees
- moved R8 267.7 mm to (275.1, 158.0), turned to 180 degrees
- moved C8 262.4 mm to (261.2, 111.2)
- moved C12 256.9 mm to (260.4, 145.5), turned to 90 degrees
- moved R4 251.2 mm to (267.2, 116.0), turned to 90 degrees
- moved C5 248.8 mm to (245.2, 105.3), turned to -90 degrees
- moved D1 245.0 mm to (263.4, 117.0), turned to 90 degrees
- moved R2 241.8 mm to (267.2, 110.9), turned to 180 degrees
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Routing:
- net GND: track 23.9 -> 67.1 mm, vias 117 -> 161
- net +12C: track 0.00 -> 22.1 mm, vias 0 -> 14
- net +12V: track 0.00 -> 22.1 mm, vias 0 -> 14
- net +12LF: track 0.00 -> 22.1 mm, vias 0 -> 14
- net +12P: track 0.00 -> 22.1 mm, vias 0 -> 14
- net Net-(IC5-ON/~{OFF}): track 0.00 -> 8.73 mm
- net Net-(IC5-FB): track 0.00 -> 7.70 mm
- net Net-(IC3-FB): track 0.00 -> 7.70 mm
- net Net-(IC4-FB): track 0.00 -> 7.70 mm
- net Net-(IC2-FB): track 0.00 -> 7.70 mm
- net Net-(IC3-CB): track 0.00 -> 4.29 mm
- net Net-(IC5-CB): track 0.00 -> 4.29 mm
- net Net-(IC2-CB): track 0.00 -> 4.29 mm
- net Net-(IC4-CB): track 0.00 -> 4.29 mm
- net unconnected-(IC5-TAB-Pad8): vias 0 -> 9
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- added copper zone on F.Cu, net +12C
- added copper zone on F.Cu, net +12LF
- added copper zone on F.Cu, net +12P
- added copper zone on F.Cu, net +12V
- added copper zone on F.Cu, net GND
- added copper zone on F.Cu, net Net-(D2-K)

Commit message: h bridge routing WIP
Parts:
- moved J2 323.4 mm to (258.3, 260.9)
- moved J1 274.0 mm to (233.2, 226.9)
- moved IC8 207.2 mm to (168.3, 188.7), turned to 90 degrees
- moved IC6 203.5 mm to (155.4, 188.7), turned to 90 degrees
- moved J9 189.1 mm to (158.8, 171.0)
- moved R33 187.3 mm to (152.4, 198.3), turned to 90 degrees
- moved R32 183.3 mm to (158.5, 198.1), turned to 90 degrees
- moved R34 182.2 mm to (148.3, 198.4), turned to 90 degrees
- moved R17 164.3 mm to (191.9, 143.9), turned to 45 degrees
- moved R16 162.2 mm to (189.5, 141.7), turned to -135 degrees
- moved R39 141.9 mm to (129.9, 174.8)
- moved C30 139.9 mm to (122.0, 184.3)
- moved C28 138.0 mm to (120.9, 175.3)
- moved R26 138.0 mm to (121.5, 152.4)
- moved R28 138.0 mm to (121.5, 159.0)
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Routing:
- net BATT_LVL: track 0.00 -> 9.80 mm, vias 0 -> 2
- net Net-(JP2-B): track 0.00 -> 3.03 mm
- net +BATT: track 0.00 -> 1.90 mm, vias 42 -> 43
- net EXTRA_A: track 11.9 -> 13.1 mm

Commit message: completed all h-bridge routing
Parts:
- moved IC9 290.4 mm to (279.0, 122.4), turned to 90 degrees
- moved R27 280.4 mm to (278.4, 159.5), turned to 180 degrees
- moved R29 280.0 mm to (281.2, 156.0)
- moved IC7 278.7 mm to (265.3, 122.4), turned to 90 degrees
- moved R31 273.2 mm to (275.9, 156.0)
- moved R41 266.3 mm to (283.2, 130.0), turned to 90 degrees
- moved R42 262.6 mm to (280.2, 130.0), turned to -90 degrees
- moved C31 262.3 mm to (272.5, 120.4), turned to -90 degrees
- moved R43 259.4 mm to (277.6, 130.0), turned to -90 degrees
- moved R35 254.9 mm to (266.7, 130.0), turned to 90 degrees
- moved R37 250.7 mm to (263.7, 130.0), turned to 90 degrees
- moved R36 248.9 mm to (261.2, 130.1), turned to 90 degrees
- moved IC11 242.1 mm to (230.4, 68.6), turned to 90 degrees
- moved IC10 227.7 mm to (216.6, 68.6), turned to 90 degrees
- moved C33 216.1 mm to (223.9, 66.6), turned to -90 degrees
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Routing:
- net Net-(IC7-IS): track 0.00 -> 73.4 mm, vias 0 -> 2
- net Net-(IC6-IS): track 0.00 -> 73.4 mm, vias 0 -> 2
- net Net-(IC10-IS): track 0.00 -> 73.4 mm, vias 0 -> 2
- net +12P: track 22.1 -> 44.2 mm, vias 14 -> 20
- net 1_IS: track 0.00 -> 16.1 mm, vias 0 -> 2
- net 2_IS: track 0.00 -> 13.7 mm, vias 0 -> 2
- net 3_IS: track 0.00 -> 12.3 mm, vias 0 -> 3
- net GND: track 67.1 -> 79.3 mm, vias 161 -> 183
- net Net-(IC6-EN): track 0.00 -> 9.35 mm
- net BATT_LVL: track 9.80 -> 19.1 mm
- net Net-(JP2-B): track 3.03 -> 12.1 mm
- net Net-(IC4-FB): track 7.70 -> 15.4 mm
- net Net-(IC6-DEN): track 0.00 -> 7.36 mm
- net Net-(IC11-IN): track 0.00 -> 4.72 mm
- net Net-(IC8-IN): track 0.00 -> 4.72 mm
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- added copper zone on B.Cu, net +12C
- added copper zone on B.Cu, net +12P
- added copper zone on B.Cu, net +12V
- added copper zone on F.Cu, net Net-(D1-K)
- added copper zone on F.Cu, net Net-(D3-K)
- added copper zone on F.Cu, net Net-(D5-K)

Commit message: completed motor port routing and added battery decals
Parts:
- added G***: LOGO, LOGO, F.Cu at (183.9, 135.0)
- added G***: LOGO, LOGO, F.Cu at (196.8, 134.8)
- added G***: LOGO, LOGO, F.Cu at (190.5, 134.9)
- added G***: LOGO, LOGO, F.Cu at (203.2, 134.9)
- added G***: LOGO, LOGO, F.Cu at (209.6, 134.9)
- moved J11 197.2 mm to (258.0, 145.6)
- moved J9 132.5 mm to (197.9, 73.2)
- moved R36 128.4 mm to (140.6, 174.0)
- moved C2 128.4 mm to (146.3, 203.0)
- moved C5 128.4 mm to (153.6, 196.1)
- moved C8 128.4 mm to (137.6, 190.2)
- moved IC2 128.4 mm to (128.5, 196.0)
- moved L2 128.4 mm to (144.5, 183.4)
- moved R2 128.4 mm to (131.6, 190.5)
- moved R27 128.4 mm to (157.7, 203.5)
- moved R29 128.4 mm to (160.5, 199.9)
- moved R31 128.4 mm to (155.3, 199.9)
- moved R4 128.4 mm to (131.6, 185.5)
- moved R43 128.4 mm to (157.0, 174.0)
- moved C10 128.4 mm to (155.7, 188.5)
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Routing:
- net GND: track 79.3 -> 75.3 mm, vias 183 -> 242
- added copper zone on F.Cu, net 1_LOUT
- added copper zone on F.Cu, net 1_ROUT
- added copper zone on F.Cu, net 2_LOUT
- added copper zone on F.Cu, net 2_ROUT
- added copper zone on F.Cu, net 3_LOUT
- added copper zone on F.Cu, net 3_ROUT

Commit message: Routing fully completed
Parts:
- added G***: LOGO, decals:ugs, F.Cu at (229.9, 119.6)
- added REF**: MountingHole_4.3mm_M4, MountingHole:MountingHole_4.3mm_M4, F.Cu at (143.0, 206.0)
- added REF**: MountingHole_4.3mm_M4, MountingHole:MountingHole_4.3mm_M4, F.Cu at (143.0, 93.2)
- added REF**: MountingHole_4.3mm_M4, MountingHole:MountingHole_4.3mm_M4, F.Cu at (256.3, 93.2)
- added REF**: MountingHole_4.3mm_M4, MountingHole:MountingHole_4.3mm_M4, F.Cu at (256.3, 206.0)
- moved JP3 224.7 mm to (133.4, 148.1), turned to 60 degrees
- moved R14 221.7 mm to (258.1, 137.1), turned to 120 degrees
- moved R20 220.1 mm to (135.1, 144.6), turned to -30 degrees
- moved R13 218.0 mm to (256.0, 138.8), turned to -60 degrees
- moved D5 216.8 mm to (136.1, 140.8), turned to -30 degrees
- moved R18 214.1 mm to (139.5, 147.1), turned to 60 degrees
- moved IC5 211.8 mm to (142.7, 152.5), turned to 150 degrees
- moved L6 207.6 mm to (139.8, 132.4), turned to 60 degrees
- moved C26 206.9 mm to (142.3, 141.8), turned to -120 degrees
- moved J5 204.0 mm to (249.4, 105.4), turned to 120 degrees
- moved J6 195.4 mm to (268.9, 127.5), turned to -60 degrees
- moved C27 188.5 mm to (149.8, 125.2), turned to -120 degrees
- moved C24 180.7 mm to (157.7, 140.6), turned to -30 degrees
- moved C25 180.6 mm to (155.4, 130.9), turned to 150 degrees
- moved R19 170.1 mm to (216.7, 143.0), turned to -60 degrees
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Routing:
- net M_EN_DEN: track 0.00 -> 296.7 mm, vias 0 -> 9
- net 2_HALL_B: track 0.00 -> 96.5 mm, vias 0 -> 3
- net 2_HALL_A: track 0.00 -> 95.7 mm, vias 0 -> 3
- net 3_HALL_B: track 0.00 -> 94.2 mm, vias 0 -> 5
- net 3_HALL_A: track 0.00 -> 87.7 mm, vias 0 -> 3
- net 1_HALL_A: track 0.00 -> 87.4 mm, vias 0 -> 1
- net 1_LPWM: track 0.00 -> 85.8 mm, vias 0 -> 2
- net 2_LPWM: track 0.00 -> 85.7 mm, vias 0 -> 4
- net 1_HALL_B: track 0.00 -> 84.0 mm, vias 0 -> 3
- net STOP: track 0.00 -> 73.7 mm, vias 0 -> 3
- net 1_RPWM: track 0.00 -> 70.4 mm, vias 0 -> 2
- net 3_LPWM: track 0.00 -> 69.2 mm, vias 0 -> 3
- net PI_TX: track 0.00 -> 68.2 mm, vias 0 -> 2
- net 2_RPWM: track 0.00 -> 65.7 mm, vias 0 -> 4
- net 3_RPWM: track 0.00 -> 63.5 mm, vias 0 -> 2
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- added copper zone on In2.Cu, net +5V
- added copper zone on B.Cu, net +BATT
Other:
- board size 200 x 200 mm -> 171 x 171 mm
- board text added: "locked"
