File: rbc_circuits.kicad_pcb (KiCad board)
At the start: 4 copper layers, 171 x 171 mm, 139 parts, among them IC1 LT8609AEDDM#PBF, IC10 BTN70301EPAXUMA1, IC11 BTN70301EPAXUMA1, IC2 LM2678SX-ADJ/NOPB, IC3 LM2678SX-ADJ/NOPB, IC4 LM2678SX-ADJ/NOPB, IC5 LM2678SX-ADJ/NOPB, IC6 BTN70301EPAXUMA1, IC7 BTN70301EPAXUMA1, IC8 BTN70301EPAXUMA1, IC9 BTN70301EPAXUMA1, J1 Conn_01x02_Pin, J10 Conn_01x06_Pin, J11 Conn_01x06_Pin, J2 Extra, J3 ICSP, J4 PROG, J5 External Switch, J6 Raspberry Pi Power/UART, J7 Extra 12V, J8 Extra 12V, J9 Conn_01x06_Pin, U1 CSTCE16M0V53-R0, U2 ATmega2560-16A

Commit message: completed BOM
Parts:
- added G***: LOGO, LOGO, B.Cu at (200.0, 150.0)
Other:
- board text added: "ロボットペニス!"
Changed lines of the file:
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@@
       (usegerberattributes true)
       (usegerberadvancedattributes true)
-      (creategerberjobfile true)
+      (creategerberjobfile false)
       (dashed_line_dash_ratio 12.000000)
       (dashed_line_gap_ratio 3.000000)
@@
       (drillshape 0)
       (scaleselection 1)
-      (outputdirectory "C:/Users/Kenneth/OneDrive/Desktop/temp file/")
+      (outputdirectory "C:/Users/Kenneth/OneDrive/Documents/GitHub/rbc-circuit-rev2/PCBA files/")
     )
   )
@@
     )
   )
+  (footprint "LOGO" (layer "B.Cu")
+    (at 200 150 180)
+    (attr board_only exclude_from_pos_files exclude_from_bom)
+    (fp_text reference "G***" (at 0 0) (layer "B.SilkS") hide
+        (effects (font (size 1.5 1.5) (thickness 0.3)) (justify mirror))
+    )
+    (fp_text value "LOGO" (at 0.75 0) (layer "B.SilkS") hide
+        (effects (font (size 1.5 1.5) (thickness 0.3)) (justify mirror))
+    )
+    (fp_poly
+      (pts
+        (xy 0.214404 9.977938)
+        (xy 0.404594 9.780216)
+        (xy 0.678643 9.424358)
+        (xy 1.049853 8.889657)
+        (xy 1.531523 8.155404)
+        (xy 2.136951 7.200889)
+        (xy 2.879438 6.005403)
+        (xy 3.772283 4.548239)
+        (xy 4.828785 2.808686)
+        (xy 6.062245 0.766037)
+        (xy 6.255224 0.445707)
+        (xy 7.301919 -1.298761)
+        (xy 8.287648 -2.954413)
+        (xy 9.19521 -4.491497)
+        (xy 10.007399 -5.880264)
+        (xy 10.707012 -7.090961)
+        (xy 11.276847 -8.093837)
+        (xy 11.699699 -8.859141)
+        (xy 11.958365 -9.357122)
+        (xy 12.036567 -9.552389)
+        (xy 12.036567 -9.951492)
+        (xy 0.136763 -10.000306)
+        (xy -2.298536 -10.009565)
+        (xy -4.382028 -10.015466)
+        (xy -6.140999 -10.017444)
+        (xy -7.602738 -10.014934)
+        (xy -8.79453 -10.007368)
+        (xy -9.743663 -9.994183)
+        (xy -10.477425 -9.974811)
+        (xy -11.023101 -9.948688)
+        (xy -11.407979 -9.915247)
+        (xy -11.659347 -9.873923)
+        (xy -11.804491 -9.82415)
+        (xy -11.870697 -9.765362)
+        (xy -11.877357 -9.75122)
+        (xy -11.805159 -9.521601)
+        (xy -11.538508 -8.981133)
+        (xy -11.52509 -8.956343)
+        (xy -10.298301 -8.956343)
+        (xy -10.096749 -8.986385)
+        (xy -9.55825 -9.012746)
+        (xy -8.724945 -9.035445)
+        (xy -7.638973 -9.054497)
+        (xy -6.342475 -9.069919)
+        (xy -4.877591 -9.081728)
+        (xy -3.286461 -9.089942)
+        (xy -1.611225 -9.094576)
+        (xy 0.105977 -9.095647)
+        (xy 1.823006 -9.093173)
+        (xy 3.49772 -9.087169)
+        (xy 5.087979 -9.077654)
+        (xy 6.551645 -9.064643)
+        (xy 7.846576 -9.048153)
+        (xy 8.930633 -9.028201)
+        (xy 9.761676 -9.004805)
+        (xy 10.297564 -8.97798)
+        (xy 10.495979 -8.948064)
+        (xy 10.43183 -8.747478)
+        (xy 10.200563 -8.282153)
+        (xy 9.834966 -7.609465)
+        (xy 9.36783 -6.786787)
+        (xy 8.831944 -5.871495)
+        (xy 8.260097 -4.920964)
+        (xy 7.68508 -3.992568)
+        (xy 7.471394 -3.655687)
+        (xy 7.203166 -3.236002)
+        (xy 6.018374 -3.975513)
+        (xy 4.146332 -4.93914)
+        (xy 2.229096 -5.529056)
+        (xy 0.285386 -5.745228)
+        (xy -1.666077 -5.587623)
+        (xy -3.606572 -5.056207)
+        (xy -5.517379 -4.150948)
+        (xy -5.778119 -3.996406)
+        (xy -7.00153 -3.253158)
+        (xy -7.43311 -3.948594)
+        (xy -8.28397 -5.332509)
+        (xy -9.006232 -6.5335)
+        (xy -9.584202 -7.524139)
+        (xy -10.002188 -8.276999)
+        (xy -10.244498 -8.764653)
+        (xy -10.298301 -8.956343)
+        (xy -11.52509 -8.956343)
+        (xy -11.083585 -8.140629)
+        (xy -10.446572 -7.010903)
+        (xy -9.633649 -5.602768)
+        (xy -8.650998 -3.927037)
+        (xy -7.802374 -2.496238)
+        (xy -6.065671 -2.496238)
+        (xy -5.905063 -2.674828)
+        (xy -5.478515 -2.959642)
+        (xy -4.868946 -3.308514)
+        (xy -4.159273 -3.679278)
+        (xy -3.432413 -4.029769)
+        (xy -2.771285 -4.317821)
+        (xy -2.258805 -4.501269)
+        (xy -2.037318 -4.544754)
+        (xy -2.029185 -4.40131)
+        (xy -2.175945 -4.034669)
+        (xy -2.274258 -3.84124)
+        (xy -2.598605 -2.89365)
+        (xy -2.596432 -1.936885)
+        (xy -2.364845 -1.251275)
+        (xy -2.192961 -0.852121)
+        (xy -2.160818 -0.621252)
+        (xy -2.166187 -0.613912)
+        (xy -2.414839 -0.604078)
+        (xy -2.903054 -0.747597)
+        (xy -3.545122 -1.003095)
+        (xy -4.255332 -1.329199)
+        (xy -4.947976 -1.684536)
+        (xy -5.537342 -2.027733)
+        (xy -5.937722 -2.317417)
+        (xy -6.065671 -2.496238)
+        (xy -7.802374 -2.496238)
+        (xy -7.5048 -1.994522)
+        (xy -6.60239 -0.486437)
+        (xy -5.307462 -0.486437)
+        (xy -5.23699 -0.561017)
+        (xy -5.08824 -0.518621)
+        (xy 2.239017 -0.518621)
+        (xy 2.541151 -1.102882)
+        (xy 2.76933 -1.83025)
+        (xy 2.822335 -2.674155)
+        (xy 2.698989 -3.4569)
+        (xy 2.558955 -3.791044)
+        (xy 2.35983 -4.17688)
+        (xy 2.281344 -4.395584)
+        (xy 2.43042 -4.435171)
+        (xy 2.838863 -4.329486)
+        (xy 3.429668 -4.10811)
+        (xy 4.125828 -3.800627)
+        (xy 4.85034 -3.436616)
+        (xy 5.023135 -3.342325)
+        (xy 5.593812 -2.991121)
+        (xy 6.002011 -2.674558)
+        (xy 6.160419 -2.460475)
+        (xy 6.160448 -2.458659)
+        (xy 6.000797 -2.267176)
+        (xy 5.580191 -1.973441)
+        (xy 4.986148 -1.624483)
+        (xy 4.306185 -1.267336)
+        (xy 3.627822 -0.94903)
+        (xy 3.038577 -0.716597)
+        (xy 2.778091 -0.641007)
+        (xy 2.239017 -0.518621)
+        (xy -5.08824 -0.518621)
+        (xy -4.981046 -0.488069)
+        (xy -4.472844 -0.24708)
+        (xy -4.388169 -0.204075)
+        (xy -2.88725 0.371087)
+        (xy -1.209161 0.690121)
+        (xy 0.544359 0.753003)
+        (xy 2.27157 0.559707)
+        (xy 3.870731 0.110208)
+        (xy 4.573404 -0.201872)
+        (xy 5.051334 -0.417275)
+        (xy 5.374838 -0.510389)
+        (xy 5.439212 -0.500091)
+        (xy 5.370427 -0.319499)
+        (xy 5.128696 0.142623)
+        (xy 4.738064 0.843896)
+        (xy 4.222576 1.741946)
+        (xy 3.606275 2.794393)
+        (xy 2.913206 3.958862)
+        (xy 2.840913 4.079321)
+        (xy 2.13471 5.24152)
+        (xy 1.487632 6.280417)
+        (xy 0.925745 7.156232)
+        (xy 0.475119 7.829187)
+        (xy 0.161822 8.2595)
+        (xy 0.011922 8.407394)
+        (xy 0.006447 8.404622)
+        (xy -0.128571 8.201662)
+        (xy -0.421757 7.730077)
+        (xy -0.842333 7.041359)
+        (xy -1.359524 6.187004)
+        (xy -1.942554 5.218504)
+        (xy -2.560647 4.187352)
+        (xy -3.183026 3.145042)
+        (xy -3.778917 2.143067)
+        (xy -4.317542 1.232921)
+        (xy -4.768126 0.466097)
+        (xy -5.099893 -0.105912)
+        (xy -5.282066 -0.431612)
+        (xy -5.307462 -0.486437)
+        (xy -6.60239 -0.486437)
+        (xy -6.201235 0.183962)
+        (xy -6.138 0.289224)
+        (xy -4.86285 2.407214)
+        (xy -3.766579 4.218027)
+        (xy -2.836445 5.741597)
+        (xy -2.059702 6.997858)
+        (xy -1.423607 8.006742)
+        (xy -0.915416 8.788183)
+        (xy -0.522386 9.362115)
+        (xy -0.231772 9.748471)
+        (xy -0.030831 9.967183)
+        (xy 0.093182 10.038186)
+        (xy 0.094776 10.038234)
+      )
+      (stroke (width 0) (type solid)) (fill solid) (layer "B.SilkS"))
+  )
   (gr_rect locked (start 177.3 116.023) (end 188.222 126.437)
     (stroke (width 0.2) (type solid)) (fill solid) (layer "B.Cu"))
@@
   (gr_circle locked (center 200 150) (end 285.5 150)
     (stroke (width 0.1) (type default)) (fill none) (layer "Edge.Cuts"))
+  (gr_text "ロボットペニス!" (at 243.84 175.768 -90) (layer "B.SilkS")
+    (effects (font (size 7 8) (thickness 0.8)) (justify left bottom mirror))
+  )
   (gr_text locked "MOTOR CONTROLLER PCB Rev 2.0" (at 187.452 191.516) (layer "F.SilkS")
     (effects (font (size 1.5 1.5) (thickness 0.3) bold) (justify left bottom))
@@
         (xy 298.61574 153.974078)
         (xy 298.675769 151.987442)
-        (xy 298.695782 150)
       )
     )
@@
         (xy 292.908047 153.842705)
         (xy 292.96762 151.921763)
-        (xy 292.987481 150)
       )
     )
